File: elfo/lfo.kicad_pcb (KiCad board)
At the start: 2 copper layers, 20 x 113 mm, 48 parts, among them J1 TRI, J2 SQR, J3 EURORACK, J4 TRI, J5 SQR, Q1 MMBT3904, Q2 MMBT3904, Q3 MMBT3906, Q4 MMBT3906, SW1 LFO1 SLOW, SW2 LFO2 SLOW, U1 TL074

Commit message: Make ELFO nicer, fix issues
Parts:
- moved C5 6.61 mm to (118.4, 38.2), turned to 90 degrees
- moved C6 5.60 mm to (101.3, 38.2), turned to 90 degrees
- moved C8 1.21 mm to (116.6, 45.2)
- moved J3 1.20 mm to (110.0, 38.2)
- moved C7 0.61 mm to (106.9, 45.2)
Routing:
- net +12V: track 117.1 -> 138.1 mm
- net GND: track 215.1 -> 195.6 mm
- net Net-(R12-Pad2): track 78.1 -> 90.7 mm
- net Net-(R14-Pad2): track 84.4 -> 76.2 mm
- net Net-(R8-Pad1): track 33.7 -> 29.7 mm
- net Net-(C3-Pad2): track 38.3 -> 34.3 mm
- net Net-(RV3-Pad2): track 45.9 -> 42.7 mm
- net Net-(R1-Pad1): track 57.5 -> 60.3 mm
- net Net-(R11-Pad2): track 43.2 -> 45.2 mm
- net Net-(C1-Pad2): track 44.4 -> 42.5 mm
- net -12V: track 116.5 -> 115.7 mm
- net Net-(D5-Pad1): track 7.96 -> 8.75 mm, vias 0 -> 2
- net Net-(Q2-Pad1): track 25.2 -> 25.7 mm
- added copper zone on B.Cu, net (none)
- added copper zone on F.Cu, net (none)
Other:
- board size 20 x 113 mm -> 20 x 109 mm
